Commit message: Cleanup: keeping only src, license, and readme

File: src/locus_description/urdf/locus_robot.urdf.xacro (robot description, xacro)
@@ -1,43 +1,34 @@
 <?xml version="1.0"?>
 <robot xmlns:xacro="http://www.ros.org/wiki/xacro" name="locus_robot">
-  <!-- ===================== PROPERTIES ===================== -->
-  <!-- Robot dimensions -->
   <xacro:property name="chassis_length" value="0.8"/>
   <xacro:property name="chassis_width"  value="0.6"/>
   <xacro:property name="chassis_height" value="0.3"/>
   <xacro:property name="chassis_mass"   value="4.0"/>
-  <!-- Wheels -->
-  <xacro:property name="wheel_radius" value="0.06"/>
-  <xacro:property name="wheel_width"  value="0.06"/>
-  <xacro:property name="wheel_mass"   value="0.175"/>
-  <!-- Layout -->
-  <xacro:property name="track_width" value="0.5"/>   <!-- left-right -->
-  <xacro:property name="wheel_base"  value="0.6"/>   <!-- front-back -->
-  <!-- ===================== INERTIA MACROS ===================== -->
+  <xacro:property name="wheel_radius"   value="0.06"/>
+  <xacro:property name="wheel_width"    value="0.06"/>
+  <xacro:property name="wheel_mass"     value="0.175"/>
+  <xacro:property name="track_width"    value="0.5"/>
+  <xacro:property name="wheel_base"     value="0.6"/>
   <xacro:macro name="box_inertia" params="m w h d">
     <inertial>
-      <origin xyz="0 0 0"/>
+      <origin xyz="0 0 0" rpy="0 0 0"/>
       <mass value="${m}"/>
-      <inertia
-        ixx="${(m/12)*(h*h + d*d)}" ixy="0" ixz="0"
-        iyy="${(m/12)*(w*w + d*d)}" iyz="0"
-        izz="${(m/12)*(w*w + h*h)}"/>
+      <inertia ixx="${(m/12)*(h*h + d*d)}" ixy="0" ixz="0"
+               iyy="${(m/12)*(w*w + d*d)}" iyz="0"
+               izz="${(m/12)*(w*w + h*h)}"/>
     </inertial>
   </xacro:macro>
   <xacro:macro name="cylinder_inertia" params="m r h">
     <inertial>
-      <origin xyz="0 0 0"/>
+      <origin xyz="0 0 0" rpy="0 0 0"/>
       <mass value="${m}"/>
-      <inertia
-        ixx="${(m/12)*(3*r*r + h*h)}" ixy="0" ixz="0"
-        iyy="${(m/12)*(3*r*r + h*h)}" iyz="0"
-        izz="${(m/2)*r*r}"/>
+      <inertia ixx="${(m/12)*(3*r*r + h*h)}" ixy="0" ixz="0"
+               iyy="${(m/12)*(3*r*r + h*h)}" iyz="0"
+               izz="${(m/2)*r*r}"/>
     </inertial>
   </xacro:macro>
-  <!-- ===================== MATERIALS ===================== -->
   <material name="blue"><color rgba="0.1 0.4 0.8 1"/></material>
   <material name="black"><color rgba="0 0 0 1"/></material>
   <material name="grey"><color rgba="0.5 0.5 0.5 1"/></material>
-  <!-- ===================== BASE FOOTPRINT ===================== -->
   <link name="base_footprint"/>
   <joint name="base_footprint_joint" type="fixed">
@@ -46,45 +37,28 @@
     <origin xyz="0 0 ${wheel_radius}"/>
   </joint>
-  <!-- ===================== CHASSIS ===================== -->
   <link name="base_link">
     <visual>
       <origin xyz="0 0 ${chassis_height/2}"/>
-      <geometry>
-        <box size="${chassis_length} ${chassis_width} ${chassis_height}"/>
-      </geometry>
+      <geometry><box size="${chassis_length} ${chassis_width} ${chassis_height}"/></geometry>
       <material name="blue"/>
     </visual>
     <collision>
       <origin xyz="0 0 ${chassis_height/2}"/>
-      <geometry>
-        <box size="${chassis_length} ${chassis_width} ${chassis_height}"/>
-      </geometry>
+      <geometry><box size="${chassis_length} ${chassis_width} ${chassis_height}"/></geometry>
     </collision>
-    <xacro:box_inertia
-      m="${chassis_mass}"
-      w="${chassis_width}"
-      h="${chassis_height}"
-      d="${chassis_length}"/>
+    <xacro:box_inertia m="${chassis_mass}" w="${chassis_width}" h="${chassis_height}" d="${chassis_length}"/>
   </link>
-  <!-- ===================== WHEEL MACRO ===================== -->
   <xacro:macro name="wheel" params="name x y">
     <link name="${name}_wheel">
       <visual>
         <origin rpy="${pi/2} 0 0"/>
-        <geometry>
-          <cylinder radius="${wheel_radius}" length="${wheel_width}"/>
-        </geometry>
+        <geometry><cylinder radius="${wheel_radius}" length="${wheel_width}"/></geometry>
         <material name="black"/>
       </visual>
       <collision>
         <origin rpy="${pi/2} 0 0"/>
-        <geometry>
-          <cylinder radius="${wheel_radius}" length="${wheel_width}"/>
-        </geometry>
+        <geometry><cylinder radius="${wheel_radius}" length="${wheel_width}"/></geometry>
       </collision>
-      <xacro:cylinder_inertia
-        m="${wheel_mass}"
-        r="${wheel_radius}"
-        h="${wheel_width}"/>
+      <xacro:cylinder_inertia m="${wheel_mass}" r="${wheel_radius}" h="${wheel_width}"/>
     </link>
     <joint name="${name}_wheel_joint" type="continuous">
@@ -95,102 +69,28 @@
     </joint>
   </xacro:macro>
-  <!-- ===================== 4 WHEELS ===================== -->
-  <!-- Front Left -->
-  <xacro:wheel name="front_left"
-               x="${wheel_base/2}"
-               y="${track_width/2}"/>
-  <!-- Front Right -->
-  <xacro:wheel name="front_right"
-               x="${wheel_base/2}"
-               y="${-track_width/2}"/>
-  <!-- Rear Left -->
-  <xacro:wheel name="rear_left"
-               x="${-wheel_base/2}"
-               y="${track_width/2}"/>
-  <!-- Rear Right -->
-  <xacro:wheel name="rear_right"
-               x="${-wheel_base/2}"
-               y="${-track_width/2}"/>
-<!-- ===================== LIDAR ===================== -->
-<link name="lidar_link">
-  <visual>
-    <geometry>
-      <cylinder radius="0.05" length="0.05"/>
-    </geometry>
-    <material name="grey"/>
-  </visual>
-  <collision>
-    <geometry>
-      <cylinder radius="0.05" length="0.05"/>
-    </geometry>
-  </collision>
-  <inertial>
-    <mass value="0.2"/>
-    <inertia ixx="0.001" ixy="0" ixz="0"
-             iyy="0.001" iyz="0" izz="0.001"/>
-  </inertial>
-</link>
-<joint name="lidar_joint" type="fixed">
-  <parent link="base_link"/>
-  <child  link="lidar_link"/>
-  <!-- top center of robot -->
-  <origin xyz="0 0 ${chassis_height + 0.02}" rpy="0 0 0"/>
-</joint>
-<!-- ===================== IMU ===================== -->
-<link name="imu_link">
-  <visual>
-    <geometry>
-      <box size="0.03 0.03 0.01"/>
-    </geometry>
-    <material name="grey"/>
-  </visual>
-  <collision>
-    <geometry>
-      <box size="0.03 0.03 0.01"/>
-    </geometry>
-  </collision>
-  <inertial>
-    <mass value="0.02"/>
-    <inertia ixx="0.0001" ixy="0" ixz="0"
-             iyy="0.0001" iyz="0" izz="0.0001"/>
-  </inertial>
-</link>
-<joint name="imu_joint" type="fixed">
-  <parent link="base_link"/>
-  <child  link="imu_link"/>
-  <!-- center of mass area -->
-  <origin xyz="0 0 ${chassis_height/2}" rpy="0 0 0"/>
-</joint>
-<!-- ===================== CAMERA ===================== -->
-<link name="camera_link">
-  <visual>
-    <geometry>
-      <box size="0.05 0.08 0.05"/>
-    </geometry>
-    <material name="grey"/>
-  </visual>
-  <collision>
-    <geometry>
-      <box size="0.05 0.08 0.05"/>
-    </geometry>
-  </collision>
-  <inertial>
-    <mass value="0.1"/>
-    <inertia ixx="0.0002" ixy="0" ixz="0"
-             iyy="0.0002" iyz="0" izz="0.0002"/>
-  </inertial>
-</link>
-<link name="camera_optical_frame"/>
-<joint name="camera_joint" type="fixed">
-  <parent link="base_link"/>
-  <child  link="camera_link"/>
-  <!-- front upper position -->
-  <origin xyz="${chassis_length/2} 0 ${chassis_height * 0.75}" rpy="0 0 0"/>
-</joint>
-<joint name="camera_optical_joint" type="fixed">
-  <parent link="camera_link"/>
-  <child  link="camera_optical_frame"/>
-  <!-- ROS optical frame convention -->
-  <origin xyz="0 0 0" rpy="${-pi/2} 0 ${-pi/2}"/>
-</joint>
+  <xacro:wheel name="front_left"  x="${wheel_base/2}"  y="${track_width/2}"/>
+  <xacro:wheel name="front_right" x="${wheel_base/2}"  y="${-track_width/2}"/>
+  <xacro:wheel name="rear_left"   x="${-wheel_base/2}" y="${track_width/2}"/>
+  <xacro:wheel name="rear_right"  x="${-wheel_base/2}" y="${-track_width/2}"/>
+  <link name="lidar_link">
+    <visual><geometry><cylinder radius="0.05" length="0.05"/></geometry><material name="grey"/></visual>
+    <collision><geometry><cylinder radius="0.05" length="0.05"/></geometry></collision>
+    <inertial><mass value="0.2"/><inertia ixx="0.001" ixy="0" ixz="0" iyy="0.001" iyz="0" izz="0.001"/></inertial>
+  </link>
+  <joint name="lidar_joint" type="fixed">
+    <parent link="base_link"/>
+    <child  link="lidar_link"/>
+    <origin xyz="0 0 ${chassis_height + 0.02}" rpy="0 0 0"/>
+  </joint>
+  <link name="imu_link">
+    <visual><geometry><box size="0.03 0.03 0.01"/></geometry><material name="grey"/></visual>
+    <collision><geometry><box size="0.03 0.03 0.01"/></geometry></collision>
+    <inertial><mass value="0.02"/><inertia ixx="0.0001" ixy="0" ixz="0" iyy="0.0001" iyz="0" izz="0.0001"/></inertial>
+  </link>
+  <joint name="imu_joint" type="fixed">
+    <parent link="base_link"/>
+    <child  link="imu_link"/>
+    <origin xyz="0 0 ${chassis_height/2}" rpy="0 0 0"/>
+  </joint>
+  <xacro:include filename="$(find locus_description)/urdf/locus_gazebo.xacro"/>
 </robot>
