Commit message: Fixed lidar Scan and IMU

File: src/locus_description/urdf/locus_gazebo.xacro (robot description, xacro)
@@ -2,8 +2,6 @@
 <robot xmlns:xacro="http://www.ros.org/wiki/xacro">
   <gazebo>
-    <!-- Differential Drive: controls all 4 wheels -->
-    <plugin
-      filename="gz-sim-diff-drive-system"
-      name="gz::sim::systems::DiffDrive">
+    <plugin filename="gz-sim-diff-drive-system"
+            name="gz::sim::systems::DiffDrive">
       <left_joint>front_left_wheel_joint</left_joint>
       <left_joint>rear_left_wheel_joint</left_joint>
@@ -19,24 +17,18 @@
       <max_wheel_acceleration>2.0</max_wheel_acceleration>
     </plugin>
-    <!-- Publishes wheel joint states to /joint_states -->
-    <plugin
-      filename="gz-sim-joint-state-publisher-system"
-      name="gz::sim::systems::JointStatePublisher">
+    <plugin filename="gz-sim-joint-state-publisher-system"
+            name="gz::sim::systems::JointStatePublisher">
       <topic>joint_states</topic>
       <update_rate>50</update_rate>
     </plugin>
-    <!-- Sensors system: required for LiDAR rendering (only ONE instance) -->
-    <plugin
-      filename="gz-sim-sensors-system"
-      name="gz::sim::systems::Sensors">
-      <render_engine>ogre</render_engine>
+    <!-- ogre2: required for gpu_lidar sensor type -->
+    <plugin filename="gz-sim-sensors-system"
+            name="gz::sim::systems::Sensors">
+      <render_engine>ogre2</render_engine>
     </plugin>
-    <!-- IMU system: required to compute IMU sensor data -->
-    <plugin
-      filename="gz-sim-imu-system"
-      name="gz::sim::systems::Imu">
+    <plugin filename="gz-sim-imu-system"
+            name="gz::sim::systems::Imu">
     </plugin>
   </gazebo>
-  <!-- LiDAR sensor: gz_frame_id removed (not valid inside sensor in Gazebo Harmonic) -->
   <gazebo reference="lidar_link">
     <sensor name="gpu_lidar" type="gpu_lidar">
@@ -46,5 +38,5 @@
         <scan>
           <horizontal>
-            <samples>640</samples>
+            <samples>360</samples>
             <resolution>1</resolution>
             <min_angle>-3.14159</min_angle>
@@ -53,12 +45,17 @@
         </scan>
         <range>
-          <min>0.1</min>
+          <min>0.15</min>
           <max>12.0</max>
         </range>
+        <noise>
+          <type>gaussian</type>
+          <mean>0.0</mean>
+          <stddev>0.01</stddev>
+        </noise>
       </lidar>
       <visualize>true</visualize>
+      <frame_id>lidar_link</frame_id>
     </sensor>
   </gazebo>
-  <!-- IMU sensor: gz_frame_id removed (not valid inside sensor in Gazebo Harmonic) -->
   <gazebo reference="imu_link">
     <sensor name="imu_sensor" type="imu">
@@ -66,7 +63,7 @@
       <update_rate>100</update_rate>
       <topic>imu</topic>
+      <frame_id>imu_link</frame_id>
     </sensor>
   </gazebo>
-  <!-- Wheel friction coefficients -->
   <gazebo reference="rear_left_wheel"><mu1>1.0</mu1><mu2>1.0</mu2></gazebo>
   <gazebo reference="rear_right_wheel"><mu1>1.0</mu1><mu2>1.0</mu2></gazebo>

File: src/locus_description/urdf/locus_robot.urdf.xacro (robot description, xacro)
@@ -73,7 +73,7 @@
   <xacro:wheel name="rear_left"   x="${-wheel_base/2}" y="${track_width/2}"/>
   <xacro:wheel name="rear_right"  x="${-wheel_base/2}" y="${-track_width/2}"/>
+  <!-- lidar_link: no collision block so laser rays are not blocked by own geometry -->
   <link name="lidar_link">
     <visual><geometry><cylinder radius="0.05" length="0.05"/></geometry><material name="grey"/></visual>
-    <collision><geometry><cylinder radius="0.05" length="0.05"/></geometry></collision>
     <inertial><mass value="0.2"/><inertia ixx="0.001" ixy="0" ixz="0" iyy="0.001" iyz="0" izz="0.001"/></inertial>
   </link>
@@ -81,9 +81,9 @@
     <parent link="base_link"/>
     <child  link="lidar_link"/>
-    <origin xyz="0 0 ${chassis_height + 0.02}" rpy="0 0 0"/>
+    <origin xyz="0 0 ${chassis_height + 0.1}" rpy="0 0 0"/>
   </joint>
+  <!-- imu_link: no collision block, it is a sensor not a physical obstacle -->
   <link name="imu_link">
     <visual><geometry><box size="0.03 0.03 0.01"/></geometry><material name="grey"/></visual>
-    <collision><geometry><box size="0.03 0.03 0.01"/></geometry></collision>
     <inertial><mass value="0.02"/><inertia ixx="0.0001" ixy="0" ixz="0" iyy="0.0001" iyz="0" izz="0.0001"/></inertial>
   </link>

Commit message: a not worknig version of pid for testing

File: src/locus_description/urdf/locus_gazebo.xacro (robot description, xacro)
@@ -2,33 +2,25 @@
 <robot xmlns:xacro="http://www.ros.org/wiki/xacro">
   <gazebo>
-    <plugin filename="gz-sim-diff-drive-system"
-            name="gz::sim::systems::DiffDrive">
-      <left_joint>front_left_wheel_joint</left_joint>
-      <left_joint>rear_left_wheel_joint</left_joint>
-      <right_joint>front_right_wheel_joint</right_joint>
-      <right_joint>rear_right_wheel_joint</right_joint>
-      <wheel_separation>${track_width}</wheel_separation>
-      <wheel_radius>${wheel_radius}</wheel_radius>
-      <topic>cmd_vel</topic>
-      <odom_topic>odom</odom_topic>
-      <frame_id>odom</frame_id>
-      <child_frame_id>base_footprint</child_frame_id>
-      <max_wheel_torque>20</max_wheel_torque>
-      <max_wheel_acceleration>2.0</max_wheel_acceleration>
+    <!-- ros2_control plugin: replaces the old DiffDrive plugin.
+         Connects Gazebo physics to the ros2_control hardware interface.
+         The actual control logic lives in the controller (see yaml config). -->
+    <plugin filename="gz_ros2_control-system"
+            name="gz_ros2_control::GazeboSimROS2ControlPlugin">
+      <parameters>$(find locus_description)/config/locus_controllers.yaml</parameters>
+      <ros>
+        <remapping>~/robot_description:=/robot_description</remapping>
+      </ros>
     </plugin>
-    <plugin filename="gz-sim-joint-state-publisher-system"
-            name="gz::sim::systems::JointStatePublisher">
-      <topic>joint_states</topic>
-      <update_rate>50</update_rate>
-    </plugin>
-    <!-- ogre2: required for gpu_lidar sensor type -->
+    <!-- Sensors system: required for LiDAR and IMU rendering -->
     <plugin filename="gz-sim-sensors-system"
             name="gz::sim::systems::Sensors">
       <render_engine>ogre2</render_engine>
     </plugin>
+    <!-- IMU system -->
     <plugin filename="gz-sim-imu-system"
             name="gz::sim::systems::Imu">
     </plugin>
   </gazebo>
+  <!-- LiDAR sensor -->
   <gazebo reference="lidar_link">
     <sensor name="gpu_lidar" type="gpu_lidar">
@@ -58,4 +50,5 @@
     </sensor>
   </gazebo>
+  <!-- IMU sensor -->
   <gazebo reference="imu_link">
     <sensor name="imu_sensor" type="imu">
@@ -66,4 +59,5 @@
     </sensor>
   </gazebo>
+  <!-- Wheel friction -->
   <gazebo reference="rear_left_wheel"><mu1>1.0</mu1><mu2>1.0</mu2></gazebo>
   <gazebo reference="rear_right_wheel"><mu1>1.0</mu1><mu2>1.0</mu2></gazebo>

File: src/locus_description/urdf/locus_robot.urdf.xacro (robot description, xacro)
@@ -93,4 +93,38 @@
     <origin xyz="0 0 ${chassis_height/2}" rpy="0 0 0"/>
   </joint>
+<!-- ============================================================
+       ROS2 CONTROL
+       Defines the hardware interface and joints that ros2_control
+       will manage. In simulation, GazeboSystem talks to Gazebo.
+       On real hardware, you replace GazeboSystem with your
+       actual motor driver interface.
+       ============================================================ -->
+  <ros2_control name="locus_robot" type="system">
+    <hardware>
+      <!-- Simulation hardware interface — talks to Gazebo Harmonic -->
+      <plugin>gz_ros2_control/GazeboSimSystem</plugin>
+    </hardware>
+    <!-- Each wheel joint needs velocity command and state interfaces -->
+    <joint name="front_left_wheel_joint">
+      <command_interface name="velocity"/>
+      <state_interface name="velocity"/>
+      <state_interface name="position"/>
+    </joint>
+    <joint name="front_right_wheel_joint">
+      <command_interface name="velocity"/>
+      <state_interface name="velocity"/>
+      <state_interface name="position"/>
+    </joint>
+    <joint name="rear_left_wheel_joint">
+      <command_interface name="velocity"/>
+      <state_interface name="velocity"/>
+      <state_interface name="position"/>
+    </joint>
+    <joint name="rear_right_wheel_joint">
+      <command_interface name="velocity"/>
+      <state_interface name="velocity"/>
+      <state_interface name="position"/>
+    </joint>
+  </ros2_control>
   <xacro:include filename="$(find locus_description)/urdf/locus_gazebo.xacro"/>
 </robot>

Commit message: IDK what is going on but let's make a checkpoint

File: src/locus_description/urdf/locus_gazebo.xacro (robot description, xacro)
@@ -59,8 +59,74 @@
     </sensor>
   </gazebo>
-  <!-- Wheel friction -->
-  <gazebo reference="rear_left_wheel"><mu1>1.0</mu1><mu2>1.0</mu2></gazebo>
-  <gazebo reference="rear_right_wheel"><mu1>1.0</mu1><mu2>1.0</mu2></gazebo>
-  <gazebo reference="front_left_wheel"><mu1>0.8</mu1><mu2>0.8</mu2></gazebo>
-  <gazebo reference="front_right_wheel"><mu1>0.8</mu1><mu2>0.8</mu2></gazebo>
+<!-- Wheel friction — Gazebo Harmonic -->
+<!-- torsional friction = 0 prevents wheels from resisting spinning in place -->
+<!-- This is the standard fix for differential drive turning issues -->
+<gazebo reference="front_left_wheel">
+  <collision>
+    <surface>
+      <friction>
+        <ode>
+          <mu>1.0</mu>
+          <mu2>1.0</mu2>
+        </ode>
+        <torsional>
+          <coefficient>0.0</coefficient>
+          <use_patch_radius>false</use_patch_radius>
+          <patch_radius>0.0</patch_radius>
+        </torsional>
+      </friction>
+    </surface>
+  </collision>
+</gazebo>
+<gazebo reference="front_right_wheel">
+  <collision>
+    <surface>
+      <friction>
+        <ode>
+          <mu>1.0</mu>
+          <mu2>1.0</mu2>
+        </ode>
+        <torsional>
+          <coefficient>0.0</coefficient>
+          <use_patch_radius>false</use_patch_radius>
+          <patch_radius>0.0</patch_radius>
+        </torsional>
+      </friction>
+    </surface>
+  </collision>
+</gazebo>
+<gazebo reference="rear_left_wheel">
+  <collision>
+    <surface>
+      <friction>
+        <ode>
+          <mu>1.0</mu>
+          <mu2>1.0</mu2>
+        </ode>
+        <torsional>
+          <coefficient>0.0</coefficient>
+          <use_patch_radius>false</use_patch_radius>
+          <patch_radius>0.0</patch_radius>
+        </torsional>
+      </friction>
+    </surface>
+  </collision>
+</gazebo>
+<gazebo reference="rear_right_wheel">
+  <collision>
+    <surface>
+      <friction>
+        <ode>
+          <mu>1.0</mu>
+          <mu2>1.0</mu2>
+        </ode>
+        <torsional>
+          <coefficient>0.0</coefficient>
+          <use_patch_radius>false</use_patch_radius>
+          <patch_radius>0.0</patch_radius>
+        </torsional>
+      </friction>
+    </surface>
+  </collision>
+</gazebo>
 </robot>

File: src/locus_description/urdf/locus_robot.urdf.xacro (robot description, xacro)
@@ -4,8 +4,8 @@
   <xacro:property name="chassis_width"  value="0.6"/>
   <xacro:property name="chassis_height" value="0.3"/>
-  <xacro:property name="chassis_mass"   value="4.0"/>
-  <xacro:property name="wheel_radius"   value="0.06"/>
+  <xacro:property name="chassis_mass"   value="1.0"/>
+  <xacro:property name="wheel_radius"   value="0.1"/>
   <xacro:property name="wheel_width"    value="0.06"/>
-  <xacro:property name="wheel_mass"     value="0.175"/>
+  <xacro:property name="wheel_mass"     value="0.35"/>
   <xacro:property name="track_width"    value="0.5"/>
   <xacro:property name="wheel_base"     value="0.6"/>
@@ -107,20 +107,32 @@
     <!-- Each wheel joint needs velocity command and state interfaces -->
     <joint name="front_left_wheel_joint">
-      <command_interface name="velocity"/>
+      <command_interface name="velocity">
+	  <param name="min">-10</param>
+	   <param name="max">10</param>
+	 </command_interface>
       <state_interface name="velocity"/>
       <state_interface name="position"/>
     </joint>
     <joint name="front_right_wheel_joint">
-      <command_interface name="velocity"/>
+      <command_interface name="velocity">
+	<param name="min">-10</param>
+    	<param name="max">10</param>
+  	</command_interface>
       <state_interface name="velocity"/>
       <state_interface name="position"/>
     </joint>
     <joint name="rear_left_wheel_joint">
-      <command_interface name="velocity"/>
+      <command_interface name="velocity">
+	 <param name="min">-10</param>
+   	 <param name="max">10</param>
+  	</command_interface>
       <state_interface name="velocity"/>
       <state_interface name="position"/>
     </joint>
     <joint name="rear_right_wheel_joint">
-      <command_interface name="velocity"/>
+      <command_interface name="velocity">
+	<param name="min">-10</param>
+ 	 <param name="max">10</param>
+ 	</command_interface>
       <state_interface name="velocity"/>
       <state_interface name="position"/>

Commit message: working version with map, odom , liadr ,imu but not turning right or left

File: src/locus_description/urdf/locus_gazebo.xacro (robot description, xacro)
@@ -2,7 +2,5 @@
 <robot xmlns:xacro="http://www.ros.org/wiki/xacro">
   <gazebo>
-    <!-- ros2_control plugin: replaces the old DiffDrive plugin.
-         Connects Gazebo physics to the ros2_control hardware interface.
-         The actual control logic lives in the controller (see yaml config). -->
+    <!-- gz_ros2_control: publishes odom TF and joint states via controllers -->
     <plugin filename="gz_ros2_control-system"
             name="gz_ros2_control::GazeboSimROS2ControlPlugin">
@@ -12,10 +10,8 @@
       </ros>
     </plugin>
-    <!-- Sensors system: required for LiDAR and IMU rendering -->
     <plugin filename="gz-sim-sensors-system"
             name="gz::sim::systems::Sensors">
       <render_engine>ogre2</render_engine>
     </plugin>
-    <!-- IMU system -->
     <plugin filename="gz-sim-imu-system"
             name="gz::sim::systems::Imu">
@@ -59,74 +55,60 @@
     </sensor>
   </gazebo>
-<!-- Wheel friction — Gazebo Harmonic -->
-<!-- torsional friction = 0 prevents wheels from resisting spinning in place -->
-<!-- This is the standard fix for differential drive turning issues -->
-<gazebo reference="front_left_wheel">
-  <collision>
-    <surface>
-      <friction>
-        <ode>
-          <mu>1.0</mu>
-          <mu2>1.0</mu2>
-        </ode>
-        <torsional>
-          <coefficient>0.0</coefficient>
-          <use_patch_radius>false</use_patch_radius>
-          <patch_radius>0.0</patch_radius>
-        </torsional>
-      </friction>
-    </surface>
-  </collision>
-</gazebo>
-<gazebo reference="front_right_wheel">
-  <collision>
-    <surface>
-      <friction>
-        <ode>
-          <mu>1.0</mu>
-          <mu2>1.0</mu2>
-        </ode>
-        <torsional>
-          <coefficient>0.0</coefficient>
-          <use_patch_radius>false</use_patch_radius>
-          <patch_radius>0.0</patch_radius>
-        </torsional>
-      </friction>
-    </surface>
-  </collision>
-</gazebo>
-<gazebo reference="rear_left_wheel">
-  <collision>
-    <surface>
-      <friction>
-        <ode>
-          <mu>1.0</mu>
-          <mu2>1.0</mu2>
-        </ode>
-        <torsional>
-          <coefficient>0.0</coefficient>
-          <use_patch_radius>false</use_patch_radius>
-          <patch_radius>0.0</patch_radius>
-        </torsional>
-      </friction>
-    </surface>
-  </collision>
-</gazebo>
-<gazebo reference="rear_right_wheel">
-  <collision>
-    <surface>
-      <friction>
-        <ode>
-          <mu>1.0</mu>
-          <mu2>1.0</mu2>
-        </ode>
-        <torsional>
-          <coefficient>0.0</coefficient>
-          <use_patch_radius>false</use_patch_radius>
-          <patch_radius>0.0</patch_radius>
-        </torsional>
-      </friction>
-    </surface>
-  </collision>
-</gazebo>
+  <!-- Wheel friction with torsional = 0 -->
+  <gazebo reference="front_left_wheel">
+    <collision>
+      <surface>
+        <friction>
+          <ode><mu>1.0</mu><mu2>1.0</mu2></ode>
+          <torsional>
+            <coefficient>0.0</coefficient>
+            <use_patch_radius>false</use_patch_radius>
+            <patch_radius>0.0</patch_radius>
+          </torsional>
+        </friction>
+      </surface>
+    </collision>
+  </gazebo>
+  <gazebo reference="front_right_wheel">
+    <collision>
+      <surface>
+        <friction>
+          <ode><mu>1.0</mu><mu2>1.0</mu2></ode>
+          <torsional>
+            <coefficient>0.0</coefficient>
+            <use_patch_radius>false</use_patch_radius>
+            <patch_radius>0.0</patch_radius>
+          </torsional>
+        </friction>
+      </surface>
+    </collision>
+  </gazebo>
+  <gazebo reference="rear_left_wheel">
+    <collision>
+      <surface>
+        <friction>
+          <ode><mu>1.0</mu><mu2>1.0</mu2></ode>
+          <torsional>
+            <coefficient>0.0</coefficient>
+            <use_patch_radius>false</use_patch_radius>
+            <patch_radius>0.0</patch_radius>
+          </torsional>
+        </friction>
+      </surface>
+    </collision>
+  </gazebo>
+  <gazebo reference="rear_right_wheel">
+    <collision>
+      <surface>
+        <friction>
+          <ode><mu>1.0</mu><mu2>1.0</mu2></ode>
+          <torsional>
+            <coefficient>0.0</coefficient>
+            <use_patch_radius>false</use_patch_radius>
+            <patch_radius>0.0</patch_radius>
+          </torsional>
+        </friction>
+      </surface>
+    </collision>
+  </gazebo>
 </robot>

File: src/locus_description/urdf/locus_robot.urdf.xacro (robot description, xacro)
@@ -73,5 +73,4 @@
   <xacro:wheel name="rear_left"   x="${-wheel_base/2}" y="${track_width/2}"/>
   <xacro:wheel name="rear_right"  x="${-wheel_base/2}" y="${-track_width/2}"/>
-  <!-- lidar_link: no collision block so laser rays are not blocked by own geometry -->
   <link name="lidar_link">
     <visual><geometry><cylinder radius="0.05" length="0.05"/></geometry><material name="grey"/></visual>
@@ -83,5 +82,4 @@
     <origin xyz="0 0 ${chassis_height + 0.1}" rpy="0 0 0"/>
   </joint>
-  <!-- imu_link: no collision block, it is a sensor not a physical obstacle -->
   <link name="imu_link">
     <visual><geometry><box size="0.03 0.03 0.01"/></geometry><material name="grey"/></visual>
@@ -93,22 +91,13 @@
     <origin xyz="0 0 ${chassis_height/2}" rpy="0 0 0"/>
   </joint>
-<!-- ============================================================
-       ROS2 CONTROL
-       Defines the hardware interface and joints that ros2_control
-       will manage. In simulation, GazeboSystem talks to Gazebo.
-       On real hardware, you replace GazeboSystem with your
-       actual motor driver interface.
-       ============================================================ -->
   <ros2_control name="locus_robot" type="system">
     <hardware>
-      <!-- Simulation hardware interface — talks to Gazebo Harmonic -->
       <plugin>gz_ros2_control/GazeboSimSystem</plugin>
     </hardware>
-    <!-- Each wheel joint needs velocity command and state interfaces -->
     <joint name="front_left_wheel_joint">
       <command_interface name="velocity">
-	  <param name="min">-10</param>
-	   <param name="max">10</param>
-	 </command_interface>
+        <param name="min">-10</param>
+        <param name="max">10</param>
+      </command_interface>
       <state_interface name="velocity"/>
       <state_interface name="position"/>
@@ -116,7 +105,7 @@
     <joint name="front_right_wheel_joint">
       <command_interface name="velocity">
-	<param name="min">-10</param>
-    	<param name="max">10</param>
-  	</command_interface>
+        <param name="min">-10</param>
+        <param name="max">10</param>
+      </command_interface>
       <state_interface name="velocity"/>
       <state_interface name="position"/>
@@ -124,7 +113,7 @@
     <joint name="rear_left_wheel_joint">
       <command_interface name="velocity">
-	 <param name="min">-10</param>
-   	 <param name="max">10</param>
-  	</command_interface>
+        <param name="min">-10</param>
+        <param name="max">10</param>
+      </command_interface>
       <state_interface name="velocity"/>
       <state_interface name="position"/>
@@ -132,7 +121,7 @@
     <joint name="rear_right_wheel_joint">
       <command_interface name="velocity">
-	<param name="min">-10</param>
- 	 <param name="max">10</param>
- 	</command_interface>
+        <param name="min">-10</param>
+        <param name="max">10</param>
+      </command_interface>
       <state_interface name="velocity"/>
       <state_interface name="position"/>
