Commit message: Ahh, The issue of turning in 4WD was not solved, so changed to 2WD diff drive, with proper Map, laser scan, IMU, odom and movement!

File: src/locus_description/urdf/locus_gazebo.xacro (robot description, xacro)
@@ -2,5 +2,5 @@
 <robot xmlns:xacro="http://www.ros.org/wiki/xacro">
   <gazebo>
-    <!-- gz_ros2_control: publishes odom TF and joint states via controllers -->
+    <!-- gz_ros2_control plugin -->
     <plugin filename="gz_ros2_control-system"
             name="gz_ros2_control::GazeboSimROS2ControlPlugin">
@@ -10,13 +10,123 @@
       </ros>
     </plugin>
+    <!-- Sensors system for LiDAR GPU rendering -->
     <plugin filename="gz-sim-sensors-system"
             name="gz::sim::systems::Sensors">
       <render_engine>ogre2</render_engine>
     </plugin>
+    <!-- IMU system -->
     <plugin filename="gz-sim-imu-system"
             name="gz::sim::systems::Imu">
     </plugin>
   </gazebo>
-  <!-- LiDAR sensor -->
+  <!-- =========================================================
+       CHASSIS — low friction so it doesn't drag on ground
+       selfCollide false prevents internal collisions
+       ========================================================= -->
+  <gazebo reference="base_link">
+    <selfCollide>false</selfCollide>
+    <mu1>0.0</mu1>
+    <mu2>0.0</mu2>
+  </gazebo>
+  <!-- =========================================================
+       LEFT WHEEL — high friction for traction, zero torsional
+       mu1 = friction in rolling direction (high = good traction)
+       mu2 = friction in lateral direction
+       torsional coefficient = 0 means no resistance to spinning in place
+       ========================================================= -->
+  <gazebo reference="left_wheel">
+    <selfCollide>false</selfCollide>
+    <collision>
+      <surface>
+        <friction>
+          <ode>
+            <mu>1.0</mu>
+            <mu2>1.0</mu2>
+            <fdir1>0 0 1</fdir1>
+            <slip1>0.0</slip1>
+            <slip2>0.0</slip2>
+          </ode>
+          <torsional>
+            <coefficient>0.0</coefficient>
+            <use_patch_radius>false</use_patch_radius>
+            <patch_radius>0.0</patch_radius>
+          </torsional>
+        </friction>
+        <contact>
+          <ode>
+            <kp>1000000.0</kp>
+            <kd>100.0</kd>
+            <max_vel>0.1</max_vel>
+            <min_depth>0.001</min_depth>
+          </ode>
+        </contact>
+      </surface>
+    </collision>
+  </gazebo>
+  <!-- =========================================================
+       RIGHT WHEEL — same settings as left
+       ========================================================= -->
+  <gazebo reference="right_wheel">
+    <selfCollide>false</selfCollide>
+    <collision>
+      <surface>
+        <friction>
+          <ode>
+            <mu>1.0</mu>
+            <mu2>1.0</mu2>
+            <fdir1>0 0 1</fdir1>
+            <slip1>0.0</slip1>
+            <slip2>0.0</slip2>
+          </ode>
+          <torsional>
+            <coefficient>0.0</coefficient>
+            <use_patch_radius>false</use_patch_radius>
+            <patch_radius>0.0</patch_radius>
+          </torsional>
+        </friction>
+        <contact>
+          <ode>
+            <kp>1000000.0</kp>
+            <kd>100.0</kd>
+            <max_vel>0.1</max_vel>
+            <min_depth>0.001</min_depth>
+          </ode>
+        </contact>
+      </surface>
+    </collision>
+  </gazebo>
+  <!-- =========================================================
+       CASTER WHEEL — near zero friction in all directions
+       This is the key to easy turning: caster has no resistance
+       ========================================================= -->
+  <gazebo reference="caster_wheel">
+    <selfCollide>false</selfCollide>
+    <collision>
+      <surface>
+        <friction>
+          <ode>
+            <mu>0.0</mu>
+            <mu2>0.0</mu2>
+          </ode>
+          <torsional>
+            <coefficient>0.0</coefficient>
+            <use_patch_radius>false</use_patch_radius>
+            <patch_radius>0.0</patch_radius>
+          </torsional>
+        </friction>
+        <contact>
+          <ode>
+            <kp>1000000.0</kp>
+            <kd>100.0</kd>
+            <max_vel>0.1</max_vel>
+            <min_depth>0.001</min_depth>
+          </ode>
+        </contact>
+      </surface>
+    </collision>
+  </gazebo>
+  <!-- =========================================================
+       LIDAR SENSOR
+       ========================================================= -->
   <gazebo reference="lidar_link">
     <sensor name="gpu_lidar" type="gpu_lidar">
@@ -46,5 +156,7 @@
     </sensor>
   </gazebo>
-  <!-- IMU sensor -->
+  <!-- =========================================================
+       IMU SENSOR
+       ========================================================= -->
   <gazebo reference="imu_link">
     <sensor name="imu_sensor" type="imu">
@@ -55,60 +167,3 @@
     </sensor>
   </gazebo>
-  <!-- Wheel friction with torsional = 0 -->
-  <gazebo reference="front_left_wheel">
-    <collision>
-      <surface>
-        <friction>
-          <ode><mu>1.0</mu><mu2>1.0</mu2></ode>
-          <torsional>
-            <coefficient>0.0</coefficient>
-            <use_patch_radius>false</use_patch_radius>
-            <patch_radius>0.0</patch_radius>
-          </torsional>
-        </friction>
-      </surface>
-    </collision>
-  </gazebo>
-  <gazebo reference="front_right_wheel">
-    <collision>
-      <surface>
-        <friction>
-          <ode><mu>1.0</mu><mu2>1.0</mu2></ode>
-          <torsional>
-            <coefficient>0.0</coefficient>
-            <use_patch_radius>false</use_patch_radius>
-            <patch_radius>0.0</patch_radius>
-          </torsional>
-        </friction>
-      </surface>
-    </collision>
-  </gazebo>
-  <gazebo reference="rear_left_wheel">
-    <collision>
-      <surface>
-        <friction>
-          <ode><mu>1.0</mu><mu2>1.0</mu2></ode>
-          <torsional>
-            <coefficient>0.0</coefficient>
-            <use_patch_radius>false</use_patch_radius>
-            <patch_radius>0.0</patch_radius>
-          </torsional>
-        </friction>
-      </surface>
-    </collision>
-  </gazebo>
-  <gazebo reference="rear_right_wheel">
-    <collision>
-      <surface>
-        <friction>
-          <ode><mu>1.0</mu><mu2>1.0</mu2></ode>
-          <torsional>
-            <coefficient>0.0</coefficient>
-            <use_patch_radius>false</use_patch_radius>
-            <patch_radius>0.0</patch_radius>
-          </torsional>
-        </friction>
-      </surface>
-    </collision>
-  </gazebo>
 </robot>

File: src/locus_description/urdf/locus_robot.urdf.xacro (robot description, xacro)
@@ -1,20 +1,34 @@
 <?xml version="1.0"?>
 <robot xmlns:xacro="http://www.ros.org/wiki/xacro" name="locus_robot">
-  <xacro:property name="chassis_length" value="0.8"/>
-  <xacro:property name="chassis_width"  value="0.6"/>
-  <xacro:property name="chassis_height" value="0.3"/>
+  <!-- =========================================================
+       ROBOT DIMENSIONS
+       chassis: 50cm long, 30cm wide, 10cm tall
+       wheels:  6cm radius, 4cm wide, 50g each
+       caster:  2.5cm radius sphere at front
+       total mass: ~1.1kg
+       ========================================================= -->
+  <xacro:property name="chassis_length" value="0.50"/>
+  <xacro:property name="chassis_width"  value="0.30"/>
+  <xacro:property name="chassis_height" value="0.10"/>
   <xacro:property name="chassis_mass"   value="1.0"/>
-  <xacro:property name="wheel_radius"   value="0.1"/>
-  <xacro:property name="wheel_width"    value="0.06"/>
-  <xacro:property name="wheel_mass"     value="0.35"/>
-  <xacro:property name="track_width"    value="0.5"/>
-  <xacro:property name="wheel_base"     value="0.6"/>
+  <xacro:property name="wheel_radius"   value="0.05"/>
+  <xacro:property name="wheel_width"    value="0.04"/>
+  <xacro:property name="wheel_mass"     value="0.05"/>
+  <!-- track_width = distance between left and right wheel centers -->
+  <xacro:property name="track_width"    value="0.30"/>
+  <!-- caster radius slightly less than wheel so robot sits level -->
+  <xacro:property name="caster_radius"  value="0.05"/>
+  <xacro:property name="caster_mass"    value="0.025"/>
+  <!-- =========================================================
+       INERTIA MACROS
+       ========================================================= -->
   <xacro:macro name="box_inertia" params="m w h d">
     <inertial>
       <origin xyz="0 0 0" rpy="0 0 0"/>
       <mass value="${m}"/>
-      <inertia ixx="${(m/12)*(h*h + d*d)}" ixy="0" ixz="0"
-               iyy="${(m/12)*(w*w + d*d)}" iyz="0"
-               izz="${(m/12)*(w*w + h*h)}"/>
+      <inertia
+        ixx="${(m/12)*(h*h + d*d)}" ixy="0" ixz="0"
+        iyy="${(m/12)*(w*w + d*d)}" iyz="0"
+        izz="${(m/12)*(w*w + h*h)}"/>
     </inertial>
   </xacro:macro>
@@ -23,66 +37,187 @@
       <origin xyz="0 0 0" rpy="0 0 0"/>
       <mass value="${m}"/>
-      <inertia ixx="${(m/12)*(3*r*r + h*h)}" ixy="0" ixz="0"
-               iyy="${(m/12)*(3*r*r + h*h)}" iyz="0"
-               izz="${(m/2)*r*r}"/>
+      <inertia
+        ixx="${(m/12)*(3*r*r + h*h)}" ixy="0" ixz="0"
+        iyy="${(m/12)*(3*r*r + h*h)}" iyz="0"
+        izz="${(m/2)*r*r}"/>
     </inertial>
   </xacro:macro>
-  <material name="blue"><color rgba="0.1 0.4 0.8 1"/></material>
-  <material name="black"><color rgba="0 0 0 1"/></material>
-  <material name="grey"><color rgba="0.5 0.5 0.5 1"/></material>
+  <xacro:macro name="sphere_inertia" params="m r">
+    <inertial>
+      <origin xyz="0 0 0" rpy="0 0 0"/>
+      <mass value="${m}"/>
+      <inertia
+        ixx="${(2/5)*m*r*r}" ixy="0" ixz="0"
+        iyy="${(2/5)*m*r*r}" iyz="0"
+        izz="${(2/5)*m*r*r}"/>
+    </inertial>
+  </xacro:macro>
+  <!-- =========================================================
+       MATERIALS
+       ========================================================= -->
+  <material name="blue">  <color rgba="0.1 0.4 0.8 1"/></material>
+  <material name="black"> <color rgba="0.0 0.0 0.0 1"/></material>
+  <material name="grey">  <color rgba="0.5 0.5 0.5 1"/></material>
+  <material name="white"> <color rgba="0.9 0.9 0.9 1"/></material>
+  <!-- =========================================================
+       BASE FOOTPRINT
+       ========================================================= -->
   <link name="base_footprint"/>
   <joint name="base_footprint_joint" type="fixed">
     <parent link="base_footprint"/>
     <child  link="base_link"/>
-    <origin xyz="0 0 ${wheel_radius}"/>
-  </joint>
+    <origin xyz="0 0 ${wheel_radius}" rpy="0 0 0"/>
+  </joint>
+  <!-- =========================================================
+       BASE LINK
+       ========================================================= -->
   <link name="base_link">
     <visual>
-      <origin xyz="0 0 ${chassis_height/2}"/>
-      <geometry><box size="${chassis_length} ${chassis_width} ${chassis_height}"/></geometry>
+      <origin xyz="0 0 ${chassis_height/2}" rpy="0 0 0"/>
+      <geometry>
+        <box size="${chassis_length} ${chassis_width} ${chassis_height}"/>
+      </geometry>
       <material name="blue"/>
     </visual>
     <collision>
-      <origin xyz="0 0 ${chassis_height/2}"/>
-      <geometry><box size="${chassis_length} ${chassis_width} ${chassis_height}"/></geometry>
-    </collision>
-    <xacro:box_inertia m="${chassis_mass}" w="${chassis_width}" h="${chassis_height}" d="${chassis_length}"/>
-  </link>
-  <xacro:macro name="wheel" params="name x y">
-    <link name="${name}_wheel">
-      <visual>
-        <origin rpy="${pi/2} 0 0"/>
-        <geometry><cylinder radius="${wheel_radius}" length="${wheel_width}"/></geometry>
-        <material name="black"/>
-      </visual>
-      <collision>
-        <origin rpy="${pi/2} 0 0"/>
-        <geometry><cylinder radius="${wheel_radius}" length="${wheel_width}"/></geometry>
-      </collision>
-      <xacro:cylinder_inertia m="${wheel_mass}" r="${wheel_radius}" h="${wheel_width}"/>
-    </link>
-    <joint name="${name}_wheel_joint" type="continuous">
-      <parent link="base_link"/>
-      <child  link="${name}_wheel"/>
-      <origin xyz="${x} ${y} ${-wheel_radius}"/>
-      <axis xyz="0 1 0"/>
-    </joint>
-  </xacro:macro>
-  <xacro:wheel name="front_left"  x="${wheel_base/2}"  y="${track_width/2}"/>
-  <xacro:wheel name="front_right" x="${wheel_base/2}"  y="${-track_width/2}"/>
-  <xacro:wheel name="rear_left"   x="${-wheel_base/2}" y="${track_width/2}"/>
-  <xacro:wheel name="rear_right"  x="${-wheel_base/2}" y="${-track_width/2}"/>
+      <origin xyz="0 0 ${chassis_height/2}" rpy="0 0 0"/>
+      <geometry>
+        <box size="${chassis_length} ${chassis_width} ${chassis_height}"/>
+      </geometry>
+    </collision>
+    <xacro:box_inertia
+      m="${chassis_mass}"
+      w="${chassis_width}"
+      h="${chassis_height}"
+      d="${chassis_length}"/>
+  </link>
+  <!-- =========================================================
+       LEFT DRIVE WHEEL
+       ========================================================= -->
+  <link name="left_wheel">
+    <visual>
+      <origin xyz="0 0 0" rpy="${pi/2} 0 0"/>
+      <geometry>
+        <cylinder radius="${wheel_radius}" length="${wheel_width}"/>
+      </geometry>
+      <material name="black"/>
+    </visual>
+    <collision>
+      <origin xyz="0 0 0" rpy="${pi/2} 0 0"/>
+      <geometry>
+        <cylinder radius="${wheel_radius}" length="${wheel_width}"/>
+      </geometry>
+    </collision>
+    <xacro:cylinder_inertia
+      m="${wheel_mass}"
+      r="${wheel_radius}"
+      h="${wheel_width}"/>
+  </link>
+  <joint name="left_wheel_joint" type="continuous">
+    <parent link="base_link"/>
+    <child  link="left_wheel"/>
+    <origin xyz="-0.10 ${track_width/2} ${-wheel_radius}" rpy="0 0 0"/>
+    <axis xyz="0 1 0"/>
+    <limit effort="1.0" velocity="10.0"/>
+    <dynamics damping="0.1" friction="0.1"/>
+  </joint>
+  <!-- =========================================================
+       RIGHT DRIVE WHEEL
+       ========================================================= -->
+  <link name="right_wheel">
+    <visual>
+      <origin xyz="0 0 0" rpy="${pi/2} 0 0"/>
+      <geometry>
+        <cylinder radius="${wheel_radius}" length="${wheel_width}"/>
+      </geometry>
+      <material name="black"/>
+    </visual>
+    <collision>
+      <origin xyz="0 0 0" rpy="${pi/2} 0 0"/>
+      <geometry>
+        <cylinder radius="${wheel_radius}" length="${wheel_width}"/>
+      </geometry>
+    </collision>
+    <xacro:cylinder_inertia
+      m="${wheel_mass}"
+      r="${wheel_radius}"
+      h="${wheel_width}"/>
+  </link>
+  <joint name="right_wheel_joint" type="continuous">
+    <parent link="base_link"/>
+    <child  link="right_wheel"/>
+    <origin xyz="-0.10 ${-track_width/2} ${-wheel_radius}" rpy="0 0 0"/>
+    <axis xyz="0 1 0"/>
+    <limit effort="1.0" velocity="10.0"/>
+    <dynamics damping="0.1" friction="0.1"/>
+  </joint>
+  <!-- =========================================================
+       CASTER WHEEL — front passive sphere
+       Using a sphere is the standard Gazebo approach for casters.
+       A sphere has uniform contact in all directions so it
+       slides freely without resisting the robot's rotation.
+       ========================================================= -->
+  <link name="caster_wheel">
+    <visual>
+      <origin xyz="0 0 0" rpy="0 0 0"/>
+      <geometry>
+        <sphere radius="${caster_radius}"/>
+      </geometry>
+      <material name="white"/>
+    </visual>
+    <collision>
+      <origin xyz="0 0 0" rpy="0 0 0"/>
+      <geometry>
+        <sphere radius="${caster_radius}"/>
+      </geometry>
+    </collision>
+    <xacro:sphere_inertia m="${caster_mass}" r="${caster_radius}"/>
+  </link>
+  <joint name="caster_wheel_joint" type="fixed">
+    <parent link="base_link"/>
+    <child  link="caster_wheel"/>
+    <!-- front of chassis, dropped so sphere touches ground -->
+    <origin xyz="0.18 0 ${-caster_radius}" rpy="0 0 0"/>
+  </joint>
+  <!-- =========================================================
+       LIDAR LINK
+       ========================================================= -->
   <link name="lidar_link">
-    <visual><geometry><cylinder radius="0.05" length="0.05"/></geometry><material name="grey"/></visual>
-    <inertial><mass value="0.2"/><inertia ixx="0.001" ixy="0" ixz="0" iyy="0.001" iyz="0" izz="0.001"/></inertial>
+    <visual>
+      <origin xyz="0 0 0" rpy="0 0 0"/>
+      <geometry>
+        <cylinder radius="0.04" length="0.04"/>
+      </geometry>
+      <material name="grey"/>
+    </visual>
+    <!-- no collision block — prevents lidar from hitting itself -->
+    <inertial>
+      <mass value="0.1"/>
+      <inertia ixx="0.001" ixy="0" ixz="0"
+               iyy="0.001" iyz="0" izz="0.001"/>
+    </inertial>
   </link>
   <joint name="lidar_joint" type="fixed">
     <parent link="base_link"/>
     <child  link="lidar_link"/>
-    <origin xyz="0 0 ${chassis_height + 0.1}" rpy="0 0 0"/>
-  </joint>
+    <origin xyz="0.05 0 ${chassis_height + 0.02}" rpy="0 0 0"/>
+  </joint>
+  <!-- =========================================================
+       IMU LINK
+       ========================================================= -->
   <link name="imu_link">
-    <visual><geometry><box size="0.03 0.03 0.01"/></geometry><material name="grey"/></visual>
-    <inertial><mass value="0.02"/><inertia ixx="0.0001" ixy="0" ixz="0" iyy="0.0001" iyz="0" izz="0.0001"/></inertial>
+    <visual>
+      <origin xyz="0 0 0" rpy="0 0 0"/>
+      <geometry>
+        <box size="0.03 0.03 0.01"/>
+      </geometry>
+      <material name="grey"/>
+    </visual>
+    <!-- no collision block -->
+    <inertial>
+      <mass value="0.01"/>
+      <inertia ixx="0.0001" ixy="0" ixz="0"
+               iyy="0.0001" iyz="0" izz="0.0001"/>
+    </inertial>
   </link>
   <joint name="imu_joint" type="fixed">
@@ -91,9 +226,12 @@
     <origin xyz="0 0 ${chassis_height/2}" rpy="0 0 0"/>
   </joint>
+  <!-- =========================================================
+       ROS2 CONTROL — only 2 drive wheels
+       ========================================================= -->
   <ros2_control name="locus_robot" type="system">
     <hardware>
       <plugin>gz_ros2_control/GazeboSimSystem</plugin>
     </hardware>
-    <joint name="front_left_wheel_joint">
+    <joint name="left_wheel_joint">
       <command_interface name="velocity">
         <param name="min">-10</param>
@@ -103,21 +241,5 @@
       <state_interface name="position"/>
     </joint>
-    <joint name="front_right_wheel_joint">
-      <command_interface name="velocity">
-        <param name="min">-10</param>
-        <param name="max">10</param>
-      </command_interface>
-      <state_interface name="velocity"/>
-      <state_interface name="position"/>
-    </joint>
-    <joint name="rear_left_wheel_joint">
-      <command_interface name="velocity">
-        <param name="min">-10</param>
-        <param name="max">10</param>
-      </command_interface>
-      <state_interface name="velocity"/>
-      <state_interface name="position"/>
-    </joint>
-    <joint name="rear_right_wheel_joint">
+    <joint name="right_wheel_joint">
       <command_interface name="velocity">
         <param name="min">-10</param>
